File: mowi/subsys_power.sch (KiCad schematic (older format))
At the start: 34 parts, among them U10 MCP1642D-ADJI/MC, U8 TPS25210ARPWR, U9 TPS630250RNC

Commit message: correction of U10
Parts:
- U10: value MCP1642D-ADJI/MC -> MCP1642D-50
Changed lines of the file:
@@
 U 1 1 6299596D
 P 5500 3400
-F 0 "U10" H 4950 3150 50  0000 C CNN
-F 1 "MCP1642D-ADJI/MC" H 4950 3050 50  0000 C CNN
+F 0 "U10" H 5050 3150 50  0000 C CNN
+F 1 "MCP1642D-50" H 5050 3050 50  0000 C CNN
 F 2 "Package_DFN_QFN:DFN-8-1EP_3x2mm_P0.5mm_EP1.75x1.45mm" H 5500 3243 50  0001 C CNN
 F 3 "https://ww1.microchip.com/downloads/en/DeviceDoc/20005253A.pdf" H 5100 3250 50  0001 C CNN
