File: mowi/subsys_usb.sch (KiCad schematic (older format))
At the start: 56 parts, among them J7 47346-1001, Q6 EMH3T2R, SW2 PTS636 SK25F SMTR LFS, SW3 PTS636 SK25F SMTR LFS, U5 USB2512B-I/M2, U6 USBLC6-2P6, U7 CP2102N-A02-GQFN24, Y1 XRCGB24M000F2P00R0

Commit message: correction of R6 and C20
Parts:
- C20: value 100n -> 4u7; footprint Capacitor_SMD:C_0402_1005Metric -> Capacitor_SMD:C_0603_1608Metric
Changed lines of the file:
@@
 AR Path="/63E505B5/63EB63AA" Ref="C20"  Part="1"
 F 0 "C20" H 1285 4809 50  0000 R CNN
-F 1 "100n" H 1285 4900 50  0000 R CNN
-F 2 "Capacitor_SMD:C_0402_1005Metric" H 1438 4750 50  0001 C CNN
+F 1 "4u7" H 1285 4900 50  0000 R CNN
+F 2 "Capacitor_SMD:C_0603_1608Metric" H 1438 4750 50  0001 C CNN
 F 3 "~" H 1400 4900 50  0001 C CNN
 F 4 "10V" H 1285 4991 50  0000 R CNN "Voltage"
