File: mowi/mowi.sch (KiCad schematic (older format))
At the start: 62 parts, among them J1 1909763-1, J2 132134, J3 MMCX-J-P-H-RA-TH1, J4 1909763-1 DNS, J5 MMCX-J-P-H-RA-TH1, J6 1909763-1 DNS, SW1 CAS-D20B1, U1 ESP32-WROVER-IE/E, U2 SN74LVC2T45DCU, U3 SN74AUP1T97DCK, U4 FEMCxxxGTT

Commit message: correction of R6 and C20
Parts:
- R6: value 100k -> 1k
Changed lines of the file:
@@
 P 3800 10650
 F 0 "R6" V 3593 10650 50  0000 C CNN
-F 1 "100k" V 3684 10650 50  0000 C CNN
+F 1 "1k" V 3684 10650 50  0000 C CNN
 F 2 "Resistor_SMD:R_0402_1005Metric" V 3730 10650 50  0001 C CNN
 F 3 "~" H 3800 10650 50  0001 C CNN

Commit message: Add files via upload
Parts:
- C8: value 100n -> 100p
Other:
- note added: "Timing Signal Level Conversion"
- note removed: "Greco timing circuitry"
Changed lines of the file:
@@
 P 12750 2000
 F 0 "C8" V 12408 2000 50  0000 C CNN
-F 1 "100n" V 12499 2000 50  0000 C CNN
+F 1 "100p" V 12499 2000 50  0000 C CNN
 F 2 "Capacitor_SMD:C_0402_1005Metric" H 12788 1850 50  0001 C CNN
 F 3 "~" H 12750 2000 50  0001 C CNN
@@
 	6650 5350 7250 5350
 Text Notes 5500 950  0    75   ~ 15
-Greco timing circuitry
+Timing Signal Level Conversion
 Wire Notes Line width 10
 	5500 5000 7500 5000
